File: mgr.sch (EAGLE design)
At the start: 41 parts, among them CN1 USB, CN2 SWD, CN3 BT, CN4 SF-MICROSD, IC1 LM2936DT-3.3, U2 LSM9DS0, U3 MPL115A, X1 16MHz, X2 32.768kHz

Commit message: initial commit
Parts:
- removed C1, C2: (no value), resistor:C-EUC0603K
- removed X1: 16MHz, IQD-Frequency-Products:CRYSTALS-NOGND-HC49
- added Q1: 8MHz, murata-filter:CSTCR6M00G53Z
- added R5, R6: 4k7, resistor:R-EU_R0603
- added R7, R8: 100k, resistor:R-EU_R0603
- added SJ2: RESET, SparkFun-Passives:JUMPER-PAD-3-NOYES_SILK
- CN3: value BT -> UART
- CN4: value SF-MICROSD -> MICRO_SD_CONNECTOR; device microsd:SF-MICROSD -> mgr_con_sd:MICRO_SD_CONNECTOR
- IC1: value LM2936DT-3.3 -> LM1117IMPX-3.3; device national-semiconductor:LM2936DT-3.3 -> lm1117:LM1117IMPX-3.3
- X2: device IQD-Frequency-Products:CRYSTALS-NOGND-WATCH-3X8 -> IQD-Frequency-Products:CRYSTALS-NOGND-CFPX-217
Connections:
- removed net BOOT0: U1G$5.BOOT0
- removed net PA9: U1G$2.PA9
- removed net PB10: U1G$3.PB10
- removed net PB2: U1G$3.PB2/BOOT1
- new net N$11: R7.2, SJ2.1
- net +3V3: now also IC1.OUT, IC1.OUT1, R2.2, R3.2, R4.2, R5.1, R6.1, R7.1, R8.1; no longer IC1.VO, LED1.C, LED2.C, LED3.C
- net +5V: now also IC1.IN, U1G$2.PA9; no longer IC1.VIN
- net GND: now also Q1.2, SJ2.3, U1G$5.BOOT0; no longer C1.2, C2.2
- net LED1: now also LED1.C, U1G$4.PC4; no longer R2.1
- net LED2: now also LED2.C, U1G$3.PB2/BOOT1; no longer R3.1
- net LED3: now also LED3.C, U1G$3.PB10; no longer R4.1
- net N$5: now also R2.1; no longer R2.2
- net N$6: now also R3.1; no longer R3.2
- net N$7: now also R4.1; no longer R4.2
- net NRST: now also SJ2.2
- net OSC_IN: now also Q1.1; no longer C2.1, X1.2
- net OSC_OUT: now also Q1.3; no longer C1.1, X1.1
- net PB6: now also R5.2
- net PB7: now also R6.2
- net SHDN: now also R8.2; no longer U1G$4.PC4
Other:
- note added: "if using I2C"
- moved on the sheet: C7, CN4, CN5, LED1, LED2, LED3, R2, R3, R4
